File: hw/technoshield/technoshield.kicad_pcb (KiCad board)
At the start: 2 copper layers, 85.9 x 99.9 mm, 49 parts, among them J1 101-00303-68-1-ND, P1 CONN_01X03, P2 Power, P3 Analog, P4 Digital, P5 Digital, Q1 MMBT2222A-7-F, SW1 SW_PUSH, SW2 SW_PUSH, SW3 SW_PUSH, SW4 SW_PUSH, SW5 SW_PUSH, SW6 SW_PUSH, U1 PDM1-S5-D15-S, U2 MCP23008, U3 MCP23008, U4 HEF4050B

Commit message: Issue #1 fixed.
Routing:
- net Net-(DS1-Pad14): track 105.5 -> 101.2 mm
Changed lines of the file:
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@@
     (links 126)
     (no_connects 0)
-    (area 104.337905 34.468999 209.860096 138.997)
+    (area 110.922999 34.468999 196.925001 134.568001)
     (thickness 1.6)
     (drawings 62)
-    (tracks 503)
+    (tracks 505)
     (zones 0)
     (modules 49)
@@
   (title_block
     (title "Technoshield - User Interface")
-    (date 2017-04-30)
+    (date 2017-05-02)
     (rev A)
     (company "Cégep La Pocatiere")
@@
   (segment (start 123.571 99.441) (end 123.571 93.218) (width 0.25) (layer B.Cu) (net 33))
   (segment (start 124.333 100.203) (end 123.571 99.441) (width 0.25) (layer B.Cu) (net 33))
+  (segment (start 113.284 62.611) (end 113.284 61.976) (width 0.25) (layer F.Cu) (net 34))
+  (segment (start 152.654 40.005) (end 154.686 37.973) (width 0.25) (layer F.Cu) (net 34))
+  (segment (start 151.765 40.005) (end 152.654 40.005) (width 0.25) (layer F.Cu) (net 34))
+  (segment (start 146.685 45.085) (end 151.765 40.005) (width 0.25) (layer F.Cu) (net 34))
+  (segment (start 130.175 45.085) (end 146.685 45.085) (width 0.25) (layer F.Cu) (net 34))
+  (segment (start 113.284 61.976) (end 130.175 45.085) (width 0.25) (layer F.Cu) (net 34))
   (segment (start 126.873 102.743) (end 124.206 102.743) (width 0.25) (layer B.Cu) (net 34) (status 10))
-  (segment (start 154.686 45.847) (end 154.686 37.973) (width 0.25) (layer F.Cu) (net 34) (status 20))
-  (segment (start 139.954 60.579) (end 154.686 45.847) (width 0.25) (layer F.Cu) (net 34))
-  (segment (start 115.316 60.579) (end 139.954 60.579) (width 0.25) (layer F.Cu) (net 34))
-  (segment (start 113.284 62.611) (end 115.316 60.579) (width 0.25) (layer F.Cu) (net 34))
   (via (at 113.284 62.611) (size 0.6) (drill 0.4) (layers F.Cu B.Cu) (net 34))
   (segment (start 112.268 63.627) (end 113.284 62.611) (width 0.25) (layer B.Cu) (net 34))
