File: hw/technoshield/technoshield.sch (KiCad schematic (older format))
At the start: 49 parts, among them J1 MicroSD, P1 Power, P2 Analog, P3 Digital, P4 Digital, P5 CONN_1, P6 CONN_1, P7 CONN_1, P8 CONN_1

Commit message: During developpment.
Parts:
- J1: footprint (none) -> Connectors_lib:MICRO_SD_HINGE_AMP
- R? (x5): value R -> 10k
Other:
- note added: "+/-15V Power Supply"
- note removed: "Pas sûr, à faire moi-même?\nPas de footprint."
Changed lines of the file:
@@
 LIBS:contrib
 LIBS:valves
+LIBS:Connectors
 LIBS:DataStorage
 LIBS:PDM1-S5-D15-S
@@
 F 0 "J1" H 8550 5500 60  0000 C CNN
 F 1 "MicroSD" H 8550 4100 60  0000 C CNN
-F 2 "" H 8850 4950 60  0000 C CNN
+F 2 "Connectors_lib:MICRO_SD_HINGE_AMP" H 8850 4950 60  0001 C CNN
 F 3 "" H 8850 4950 60  0000 C CNN
 	1    8750 4800
 	1    0    0    -1
 $EndComp
-Text Notes 8550 3950 0    60   ~ 0
-Pas sûr, à faire moi-même?\nPas de footprint.
 $Comp
 L MCP23008 U?
@@
 P 4150 5100
 F 0 "R?" V 4230 5100 50  0000 C CNN
-F 1 "R" V 4150 5100 50  0000 C CNN
+F 1 "10k" V 4150 5100 50  0000 C CNN
 F 2 "" V 4080 5100 50  0000 C CNN
 F 3 "" H 4150 5100 50  0000 C CNN
@@
 P 4000 5100
 F 0 "R?" V 4080 5100 50  0000 C CNN
-F 1 "R" V 4000 5100 50  0000 C CNN
+F 1 "10k" V 4000 5100 50  0000 C CNN
 F 2 "" V 3930 5100 50  0000 C CNN
 F 3 "" H 4000 5100 50  0000 C CNN
@@
 P 3850 5100
 F 0 "R?" V 3930 5100 50  0000 C CNN
-F 1 "R" V 3850 5100 50  0000 C CNN
+F 1 "10k" V 3850 5100 50  0000 C CNN
 F 2 "" V 3780 5100 50  0000 C CNN
 F 3 "" H 3850 5100 50  0000 C CNN
@@
 P 3700 5100
 F 0 "R?" V 3780 5100 50  0000 C CNN
-F 1 "R" V 3700 5100 50  0000 C CNN
+F 1 "10k" V 3700 5100 50  0000 C CNN
 F 2 "" V 3630 5100 50  0000 C CNN
 F 3 "" H 3700 5100 50  0000 C CNN
@@
 P 3550 5100
 F 0 "R?" V 3630 5100 50  0000 C CNN
-F 1 "R" V 3550 5100 50  0000 C CNN
+F 1 "10k" V 3550 5100 50  0000 C CNN
 F 2 "" V 3480 5100 50  0000 C CNN
 F 3 "" H 3550 5100 50  0000 C CNN
@@
 	1    0    0    -1
 $EndComp
+Text Notes 1950 3350 0    60   ~ 0
++/-15V Power Supply
 $EndSCHEMATC

Commit message: During developpment.
Parts:
- added C4: 0.1uF, symbol C
- added D4: Led_Small, symbol Led_Small
- added JP5, JP6: JUMPER, Pin_Headers:Pin_Header_Angled_1x02, symbol JUMPER
- added R16: R, symbol R
- JP1, JP2, JP3, JP4: renamed from JP?; footprint (none) -> Pin_Headers:Pin_Header_Angled_1x02
- P9: renamed from P?; footprint (none) -> Pin_Headers:Pin_Header_Straight_1x03
- R1, R10, R2, R3, R4, R5, R6, R7, R8, R9: renamed from R?; footprint (none) -> Resistors_SMD:R_1210_HandSoldering
- gave numbers to parts that had none: 24
Connections:
- wire segments 149 -> 176
- no-connect marks 14 -> 20
Other:
- note added: "Digikey #: 101-00303-68-1-ND"
- moved on the sheet: C1, C2, C3, C5, C6, J1, JP1, JP2, JP3, JP4, R1, R14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

Commit message: During dev.
Parts:
- C1, C2, C3, C4, C5, C6: footprint (none) -> Capacitors_THT:C_Disc_D3.0mm_W1.6mm_P2.50mm
- D1, D2, D3, D4: footprint (none) -> T67K:T67K
- RV1: symbol POT -> POT-RESCUE-technoshield
- SW1, SW2, SW3, SW4, SW5: footprint (none) -> smt_btn:smt_btn
- U1: footprint MODULE -> Connectors_lib:MICRO_SD_HINGE_AMP
- U2, U3: symbol MCP23008 -> MCP23008-RESCUE-technoshield
- U4: footprint MODULE -> SO16-3_9mm:SO16-3_9mm
Changed lines of the file:
@@
 EESchema Schematic File Version 2
-LIBS:MCP23008
+LIBS:technoshield-rescue
 LIBS:power
 LIBS:device
@@
 LIBS:contrib
 LIBS:valves
-LIBS:Connectors
 LIBS:DataStorage
 LIBS:PDM1-S5-D15-S
 LIBS:HEF4050B
+LIBS:MCP23008
+LIBS:Connectors
 LIBS:technoshield-cache
 EELAYER 25 0
@@
 $EndComp
 $Comp
-L MCP23008 U2
+L MCP23008-RESCUE-technoshield U2
 U 1 1 582F2BD1
 P 2700 6250
@@
 $EndComp
 $Comp
-L MCP23008 U3
+L MCP23008-RESCUE-technoshield U3
 U 1 1 582F2CB1
 P 2750 1800
@@
 F 0 "C3" H 6825 3300 50  0000 L CNN
 F 1 "0.1uF" H 6825 3100 50  0000 L CNN
-F 2 "" H 6838 3050 50  0001 C CNN
+F 2 "Capacitors_THT:C_Disc_D3.0mm_W1.6mm_P2.50mm" H 6838 3050 50  0001 C CNN
 F 3 "" H 6800 3200 50  0000 C CNN
 	1    6800 3200
@@
 $EndComp
 $Comp
-L POT RV1
+L POT-RESCUE-technoshield RV1
 U 1 1 582F70D7
 P 3500 3000
@@
 F 0 "D1" H 4750 6925 50  0000 L CNN
 F 1 "Led_Small" H 4625 6700 50  0000 L CNN
-F 2 "" V 4800 6800 50  0001 C CNN
+F 2 "T67K:T67K" V 4800 6800 50  0001 C CNN
 F 3 "" V 4800 6800 50  0000 C CNN
 	1    4800 6800
@@
 F 0 "D2" H 4750 7225 50  0000 L CNN
 F 1 "Led_Small" H 4625 7000 50  0000 L CNN
-F 2 "" V 4800 7100 50  0001 C CNN
+F 2 "T67K:T67K" V 4800 7100 50  0001 C CNN
 F 3 "" V 4800 7100 50  0000 C CNN
 	1    4800 7100
@@
 F 0 "D3" H 4750 7525 50  0000 L CNN
 F 1 "Led_Small" H 4625 7300 50  0000 L CNN
-F 2 "" V 4800 7400 50  0001 C CNN
+F 2 "T67K:T67K" V 4800 7400 50  0001 C CNN
 F 3 "" V 4800 7400 50  0000 C CNN
 	1    4800 7400
@@
 F 0 "SW1" H 4900 5560 50  0000 C CNN
 F 1 "SW_PUSH" H 4750 5370 50  0000 C CNN
-F 2 "" H 4750 5450 50  0001 C CNN
+F 2 "smt_btn:smt_btn" H 4750 5450 50  0001 C CNN
 F 3 "" H 4750 5450 50  0000 C CNN
 	1    4750 5450
@@
 F 0 "SW2" H 4900 5810 50  0000 C CNN
 F 1 "SW_PUSH" H 4750 5620 50  0000 C CNN
-F 2 "" H 4750 5700 50  0001 C CNN
+F 2 "smt_btn:smt_btn" H 4750 5700 50  0001 C CNN
 F 3 "" H 4750 5700 50  0000 C CNN
 	1    4750 5700
@@
 F 0 "SW3" H 4900 6060 50  0000 C CNN
 F 1 "SW_PUSH" H 4750 5870 50  0000 C CNN
-F 2 "" H 4750 5950 50  0001 C CNN
+F 2 "smt_btn:smt_btn" H 4750 5950 50  0001 C CNN
 F 3 "" H 4750 5950 50  0000 C CNN
 	1    4750 5950
@@
 F 0 "SW4" H 4900 6310 50  0000 C CNN
 F 1 "SW_PUSH" H 4750 6120 50  0000 C CNN
-F 2 "" H 4750 6200 50  0001 C CNN
+F 2 "smt_btn:smt_btn" H 4750 6200 50  0001 C CNN
 F 3 "" H 4750 6200 50  0000 C CNN
 	1    4750 6200
@@
 F 0 "SW5" H 4900 6560 50  0000 C CNN
 F 1 "SW_PUSH" H 4750 6370 50  0000 C CNN
-F 2 "" H 4750 6450 50  0001 C CNN
+F 2 "smt_btn:smt_btn" H 4750 6450 50  0001 C CNN
 F 3 "" H 4750 6450 50  0000 C CNN
 	1    4750 6450
@@
 	4450 5950 4400 5950
 Wire Wire Line
-	4400 6150 4400 5950
-Wire Wire Line
-	3450 6150 4400 6150
+	4400 5950 4400 6150
+Wire Wire Line
+	4400 6150 3450 6150
 Wire Wire Line
 	4450 5700 4350 5700
 Wire Wire Line
-	4350 6050 4350 5700
-Wire Wire Line
-	3450 6050 4350 6050
+	4350 5700 4350 6050
+Wire Wire Line
+	4350 6050 3450 6050
 Wire Wire Line
 	4450 5450 4300 5450
 Wire Wire Line
-	4300 5950 4300 5450
-Wire Wire Line
-	3450 5950 4300 5950
+	4300 5450 4300 5950
+Wire Wire Line
+	4300 5950 3450 5950
 Wire Wire Line
 	3550 5250 3550 5950
@@
 F 0 "U1" H 2350 3750 50  0000 C CNN
 F 1 "PDM1-S5-D15-S" H 2350 4200 50  0000 C CNN
-F 2 "MODULE" H 2350 3850 50  0001 C CNN
+F 2 "Connectors_lib:MICRO_SD_HINGE_AMP" H 2350 3850 50  0001 C CNN
 F 3 "DOCUMENTATION" H 2350 3850 50  0001 C CNN
 	1    2350 3850
@@
 F 0 "C5" H 7225 3300 50  0000 L CNN
 F 1 "0.1uF" H 7225 3100 50  0000 L CNN
-F 2 "" H 7238 3050 50  0001 C CNN
+F 2 "Capacitors_THT:C_Disc_D3.0mm_W1.6mm_P2.50mm" H 7238 3050 50  0001 C CNN
 F 3 "" H 7200 3200 50  0000 C CNN
 	1    7200 3200
@@
 F 0 "C6" H 7625 3300 50  0000 L CNN
 F 1 "0.1uF" H 7625 3100 50  0000 L CNN
-F 2 "" H 7638 3050 50  0001 C CNN
+F 2 "Capacitors_THT:C_Disc_D3.0mm_W1.6mm_P2.50mm" H 7638 3050 50  0001 C CNN
 F 3 "" H 7600 3200 50  0000 C CNN
 	1    7600 3200
@@
 F 0 "C2" H 6475 3950 50  0000 L CNN
 F 1 "0.1uF" H 6475 3750 50  0000 L CNN
-F 2 "" H 6488 3700 50  0001 C CNN
+F 2 "Capacitors_THT:C_Disc_D3.0mm_W1.6mm_P2.50mm" H 6488 3700 50  0001 C CNN
 F 3 "" H 6450 3850 50  0000 C CNN
 	1    6450 3850
@@
 F 0 "C1" H 6475 3300 50  0000 L CNN
 F 1 "0.1uF" H 6475 3100 50  0000 L CNN
-F 2 "" H 6488 3050 50  0001 C CNN
+F 2 "Capacitors_THT:C_Disc_D3.0mm_W1.6mm_P2.50mm" H 6488 3050 50  0001 C CNN
 F 3 "" H 6450 3200 50  0000 C CNN
 	1    6450 3200
@@
 F 0 "U4" H 7800 4950 50  0000 C CNN
 F 1 "HEF4050B" H 7800 5150 50  0000 C CNN
-F 2 "MODULE" H 7800 5050 50  0001 C CNN
+F 2 "SO16-3_9mm:SO16-3_9mm" H 7800 5050 50  0001 C CNN
 F 3 "DOCUMENTATION" H 7800 5050 50  0001 C CNN
 	1    7800 5050
@@
 F 0 "D4" H 8800 4575 50  0000 L CNN
 F 1 "Led_Small" H 8675 4350 50  0000 L CNN
-F 2 "" V 8850 4450 50  0001 C CNN
+F 2 "T67K:T67K" V 8850 4450 50  0001 C CNN
 F 3 "" V 8850 4450 50  0000 C CNN
 	1    8850 4450
@@
 F 0 "C4" H 6825 3950 50  0000 L CNN
 F 1 "0.1uF" H 6825 3750 50  0000 L CNN
-F 2 "" H 6838 3700 50  0001 C CNN
+F 2 "Capacitors_THT:C_Disc_D3.0mm_W1.6mm_P2.50mm" H 6838 3700 50  0001 C CNN
 F 3 "" H 6800 3850 50  0000 C CNN
 	1    6800 3850

Commit message: During dev PCB.
Parts:
- removed P5, P6, P7, P8: CONN_1, Socket_Arduino_Uno:Arduino_1pin, symbol CONN_1
- removed Q1: Q_NPN_BCE, symbol Q_NPN_BCE
- removed R10, R5, R6, R8, R9: 10k, Resistors_SMD:R_1210_HandSoldering, symbol R
- added Q1: MMBT2222A-7-F, TO_SOT_Packages_SMD:SOT-23, symbol Q_NPN_BEC
- added SW6: SW_PUSH, smt_btn:smt_btn, symbol SW_PUSH
- D1: value Led_Small -> LS T67K-J1K2-1-Z
- D2: value Led_Small -> LY T67K-J2L1-26-Z
- D3, D4: value Led_Small -> LP T67K-E1F2-25-Z
- J1: value MicroSD -> 101-00303-68-1-ND
- JP1, JP2, JP3, JP4, JP5, JP6: footprint Pin_Headers:Pin_Header_Angled_1x02 -> Pin_Headers:Pin_Header_Straight_1x02_Pitch2.54mm
- P1: renamed from P9; footprint Pin_Headers:Pin_Header_Straight_1x03 -> Pin_Headers:Pin_Header_Straight_1x03_Pitch2.54mm
- R1, R2, R3, R4, R7: footprint Resistors_SMD:R_1210_HandSoldering -> Resistors_THT:R_Axial_DIN0204_L3.6mm_D1.6mm_P7.62mm_Horizontal
- R11, R12, R13: value R -> 1.6k; footprint (none) -> Resistors_THT:R_Axial_DIN0204_L3.6mm_D1.6mm_P7.62mm_Horizontal
- R14, R15: footprint (none) -> Resistors_THT:R_Axial_DIN0204_L3.6mm_D1.6mm_P7.62mm_Horizontal
- R16: value R -> 750; footprint (none) -> Resistors_THT:R_Axial_DIN0204_L3.6mm_D1.6mm_P7.62mm_Horizontal
- RV1: footprint (none) -> POTENTIOMETRES:POTENTIOMETRE_BOURNS_3319P
- U1: footprint Connectors_lib:MICRO_SD_HINGE_AMP -> PDM1-S:PDM1-S
- renumbered P1 to P2, P2 to P3, P3 to P4, P4 to P5
Connections:
- wire segments 176 -> 165
- no-connect marks 20 -> 16
Other:
- note added: "DIGIKEY #: 3319P-1-103"
- note added: "Green @ 2 mA @ 1.8 V"
- note added: "Micro SD"
- note added: "Red @ 2 mA @ 1.8 V"
- note added: "Yellow @ 2 mA @ 1.8 V"
- note removed: "Ajouter pour l'alimentation des composants\n"
- note removed: "Digikey #: 101-00303-68-1-ND"
- note removed: "Holes"
- note removed: "Vérifier pour le bon pinout du BJT"
- moved on the sheet: D1, D2, D3, JP1, JP3, R1, R11, R12, R13, R3, SW1, SW2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

Commit message: Gerber done.
Parts:
- C1, SW6: supplier (none) -> Cégep
- D1: manufacturer (none) -> OSRAM Opto Semiconductors Inc.; order (none) -> 475-1180-1-ND; supplier (none) -> Digikey
- D2: manufacturer (none) -> OSRAM Opto Semiconductors Inc.; order (none) -> 475-2798-1-ND; supplier (none) -> Digikey
- D3: manufacturer (none) -> OSRAM Opto Semiconductors Inc.; order (none) -> 475-2752-1-ND; supplier (none) -> Digikey
- D4: manufacturer (none) -> OSRAM Opto Semiconductors Inc.; order (none) -> LP T67K-E1F2-25-Z; supplier (none) -> Digiey
- DS1: order (none) -> DLC01602B; supplier (none) -> Elecrow
- J1: value 101-00303-68-1-ND -> 101-00303-68; manufacturer (none) -> Amphenol Commercial Products; order (none) -> 101-00303-68-1-ND; supplier (none) -> Digikey
- Q1: manufacturer (none) -> Diodes Incorporated; order (none) -> MMBT2222A-FDICT-ND; supplier (none) -> Digikey
- RV1: manufacturer (none) -> Bourns Inc.; order (none) -> 3319P-1-103; supplier (none) -> Digikey
- U1: manufacturer (none) -> CUI Inc.; order (none) -> 102-2721-ND; supplier (none) -> Digikey
- U2, U3: manufacturer (none) -> Microchip; order (none) -> MCP23008-E/P-ND; supplier (none) -> Digikey
- U4: manufacturer (none) -> NXP; order (none) -> 568-8234-2-ND; supplier (none) -> Digiey
Other:
- note removed: "DIGIKEY #: 3319P-1-103"
Changed lines of the file:
@@
 Rev "--"
 Comp "Cégep de La Pocatière"
-Comment1 "https://creativecommons.org/licenses/by-sa/4.0/"
-Comment2 "Released under the Creative Commons Attribution Share-Alike 4.0 License"
-Comment3 "Jean-Sébastien Castonguay"
-Comment4 ""
+Comment1 "Adapted from https://learn.adafruit.com/i2c-spi-lcd-backpack"
+Comment2 "https://creativecommons.org/licenses/by-sa/4.0/"
+Comment3 "Released under the Creative Commons Attribution Share-Alike 4.0 License"
+Comment4 "Copyright 2017 Jean-Sébastien Castonguay"
 $EndDescr
 $Comp
@@
 F 2 "Displays:WC1602A" H 4450 2100 50  0000 C CIN
 F 3 "" H 4450 2150 50  0000 C CNN
+F 4 "DLC01602B" H 4450 2150 60  0001 C CNN "order"
+F 5 "Elecrow" H 4450 2150 60  0001 C CNN "supplier"
 	1    4450 2150
 	0    1    -1   0
@@
 P 9450 5250
 F 0 "J1" H 9250 5950 60  0000 C CNN
-F 1 "101-00303-68-1-ND" H 9150 4550 60  0000 C CNN
+F 1 "101-00303-68" H 9150 4550 60  0000 C CNN
 F 2 "Connectors_lib:MICRO_SD_HINGE_AMP" H 9550 5400 60  0001 C CNN
 F 3 "" H 9550 5400 60  0000 C CNN
+F 4 "101-00303-68-1-ND" H 9450 5250 60  0001 C CNN "order"
+F 5 "Amphenol Commercial Products" H 9450 5250 60  0001 C CNN "manufacturer"
+F 6 "Digikey" H 9450 5250 60  0001 C CNN "supplier"
 	1    9450 5250
 	-1   0    0    -1
@@
 F 2 "Housings_DIP:DIP-18_W7.62mm_LongPads" H 2950 5950 50  0001 C CNN
 F 3 "http://ww1.microchip.com/downloads/en/DeviceDoc/21919e.pdf" H 2950 5950 50  0001 C CNN
+F 4 "MCP23008-E/P-ND" H 2950 5950 60  0001 C CNN "order"
+F 5 "Microchip" H 2950 5950 60  0001 C CNN "manufacturer"
+F 6 "Digikey" H 2950 5950 60  0001 C CNN "supplier"
 	1    2950 5950
 	1    0    0    -1
@@
 F 2 "Housings_DIP:DIP-18_W7.62mm_LongPads" H 2750 1800 50  0001 C CNN
 F 3 "http://ww1.microchip.com/downloads/en/DeviceDoc/21919e.pdf" H 2750 1800 50  0001 C CNN
+F 4 "MCP23008-E/P-ND" H 2750 1800 60  0001 C CNN "order"
+F 5 "Microchip" H 2750 1800 60  0001 C CNN "manufacturer"
+F 6 "Digikey" H 2750 1800 60  0001 C CNN "supplier"
 	1    2750 1800
 	1    0    0    -1
@@
 F 2 "POTENTIOMETRES:POTENTIOMETRE_BOURNS_3319P" H 3500 3000 50  0001 C CNN
 F 3 "" H 3500 3000 50  0000 C CNN
+F 4 "3319P-1-103" H 3500 3000 60  0001 C CNN "order"
+F 5 "Bourns Inc." H 3500 3000 60  0001 C CNN "manufacturer"
+F 6 "Digikey" H 3500 3000 60  0001 C CNN "supplier"
 	1    3500 3000
 	0    1    1    0
@@
 F 2 "T67K:T67K" V 5050 6500 50  0001 C CNN
 F 3 "" V 5050 6500 50  0000 C CNN
+F 4 "475-1180-1-ND" H 5050 6500 60  0001 C CNN "order"
+F 5 "OSRAM Opto Semiconductors Inc." H 5050 6500 60  0001 C CNN "manufacturer"
+F 6 "Digikey" H 5050 6500 60  0001 C CNN "supplier"
 	1    5050 6500
 	-1   0    0    1
@@
 F 2 "T67K:T67K" V 5050 6800 50  0001 C CNN
 F 3 "" V 5050 6800 50  0000 C CNN
+F 4 "475-2798-1-ND" H 5050 6800 60  0001 C CNN "order"
+F 5 "OSRAM Opto Semiconductors Inc." H 5050 6800 60  0001 C CNN "manufacturer"
+F 6 "Digikey" H 5050 6800 60  0001 C CNN "supplier"
 	1    5050 6800
 	-1   0    0    1
@@
 F 2 "T67K:T67K" V 5050 7100 50  0001 C CNN
 F 3 "" V 5050 7100 50  0000 C CNN
+F 4 "475-2752-1-ND" H 5050 7100 60  0001 C CNN "order"
+F 5 "OSRAM Opto Semiconductors Inc." H 5050 7100 60  0001 C CNN "manufacturer"
+F 6 "Digikey" H 5050 7100 60  0001 C CNN "supplier"
 	1    5050 7100
 	-1   0    0    1
@@
 F 2 "PDM1-S:PDM1-S" H 2350 3850 50  0001 C CNN
 F 3 "DOCUMENTATION" H 2350 3850 50  0001 C CNN
+F 4 "102-2721-ND" H 2350 3850 60  0001 C CNN "order"
+F 5 "CUI Inc." H 2350 3850 60  0001 C CNN "manufacturer"
+F 6 "Digikey" H 2350 3850 60  0001 C CNN "supplier"
 	1    2350 3850
 	1    0    0    -1
@@
 F 2 "Capacitors_THT:C_Disc_D3.0mm_W1.6mm_P2.50mm" H 6488 3050 50  0001 C CNN
 F 3 "" H 6450 3200 50  0000 C CNN
+F 4 "Cégep" H 6450 3200 60  0001 C CNN "supplier"
 	1    6450 3200
 	1    0    0    -1
@@
 F 2 "SO16-3_9mm:SO16-3_9mm" H 7800 5050 50  0001 C CNN
 F 3 "DOCUMENTATION" H 7800 5050 50  0001 C CNN
+F 4 "568-8234-2-ND" H 7800 5050 60  0001 C CNN "order"
+F 5 "NXP" H 7800 5050 60  0001 C CNN "manufacturer"
+F 6 "Digiey" H 7800 5050 60  0001 C CNN "supplier"
 	1    7800 5050
 	1    0    0    -1
@@
 F 2 "T67K:T67K" V 8850 4450 50  0001 C CNN
 F 3 "" V 8850 4450 50  0000 C CNN
+F 4 "LP T67K-E1F2-25-Z" H 8850 4450 60  0001 C CNN "order"
+F 5 "OSRAM Opto Semiconductors Inc." H 8850 4450 60  0001 C CNN "manufacturer"
+F 6 "Digiey" H 8850 4450 60  0001 C CNN "supplier"
 	1    8850 4450
 	0    -1   -1   0
@@
 Text Notes 8700 4550 1    60   ~ 0
 Green @ 2 mA @ 1.8 V
-Text Notes 3350 3450 1    60   ~ 0
-DIGIKEY #: 3319P-1-103
 $Comp
 L Q_NPN_BEC Q1
@@
 F 2 "TO_SOT_Packages_SMD:SOT-23" H 4600 1000 50  0001 C CNN
 F 3 "" H 4400 900 50  0000 C CNN
+F 4 "MMBT2222A-FDICT-ND" H 4400 900 60  0001 C CNN "order"
+F 5 "Diodes Incorporated" H 4400 900 60  0001 C CNN "manufacturer"
+F 6 "Digikey" H 4400 900 60  0001 C CNN "supplier"
 	1    4400 900
 	1    0    0    -1
@@
 F 2 "smt_btn:smt_btn" H 6600 1650 50  0001 C CNN
 F 3 "" H 6600 1650 50  0000 C CNN
+F 4 "Cégep" H 6600 1650 60  0001 C CNN "supplier"
 	1    6600 1650
 	0    -1   -1   0
